Commit message: final gpg_urdf

File: gpg_urdf/urdf/gpg.urdf (robot description, URDF)
Before this commit: robot GoPiGo3, 5 links, 4 joints
Links:
- link base_link: mass 1.0 -> None
- link camera_link: mass 0.15 -> 0.000005; geometry collision box size=0.05 0.07 0.007; visual box size=0.05 0.08 0.007
- link counter_weight: mass 0.5 -> 3; geometry collision sphere radius=0.02; visual sphere radius=0.02
- link left_wheel: mass 1.0 -> 2; geometry collision cylinder length=0.015 radius=0.0375; visual cylinder length=0.015 radius=0.0375
- link right_wheel: mass 1.0 -> 2; geometry collision cylinder length=0.015 radius=0.0375; visual cylinder length=0.015 radius=0.0375
Joints:
- removed joint counter_weight_to_base_link
- added joint ball: type fixed, parent base_link, child counter_weight, origin xyz=-0.06 0 0.0175
- joint camera_link_to_base_link: axis 0.0 1.0 0.0 -> 0 -1 0; limit lower=-0.5235 upper=0.5235 effort=300 velocity=1 -> lower=-25.00 upper=25.00 effort=1000.0 velocity=1.0; origin xyz=0.075 0.0 0.065 rpy=-1.57075 0.0 -1.57075 -> xyz=0.075 0 0.085 rpy=-1.57075 0 -1.57075 
- joint left_wheel_to_base_link: axis 1.0 0.0 0.0 -> 0 1 0; limit lower=0.0 upper=6.28 effort=300 velocity=1 -> (none); origin xyz= 0.0 -0.085 0.0375 rpy=0.0 0.0 0.0 -> xyz=0 0.075 0.035; type revolute -> continuous
- joint right_wheel_to_base_link: axis 1.0 0.0 0.0 -> 0 1 0; limit lower=0.0 upper=6.28 effort=300 velocity=1 -> (none); origin xyz=0.0 0.085 0.0375 rpy=0.0 0.0 0.0 -> xyz=0 -0.075 0.035; type revolute -> continuous
